File: extras/schematic/LCD16x02_ENCODER_CIRCUIT.sch (EAGLE design)
At the start: 12 parts, among them M1 ARDUINO-PRO-MINI-3.3V, X1 HD44780LCD-1602

Commit message: Documentation
Connections:
- net VCC: no longer M1.VCC
Other:
- note added: "3.3V"
Changed lines of the file:
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@@
 <text x="157.48" y="91.44" size="1.778" layer="91">RDA5807 module</text>
 <text x="-7.62" y="66.04" size="1.778" layer="91">Encoder</text>
+<text x="137.16" y="73.66" size="1.778" layer="91">3.3V</text>
 </plain>
 <instances>
@@
 <net name="VCC" class="0">
 <segment>
-<pinref part="M1" gate="G$1" pin="VCC"/>
 <pinref part="SUPPLY2" gate="G$1" pin="VCC"/>
-<wire x1="106.68" y1="71.12" x2="127" y2="71.12" width="0.1524" layer="91"/>
 <pinref part="U$1" gate="G$1" pin="VCC"/>
 <wire x1="153.48" y1="74.9" x2="153.48" y2="71.12" width="0.1524" layer="91"/>
 <wire x1="153.48" y1="71.12" x2="127" y2="71.12" width="0.1524" layer="91"/>
-<junction x="127" y="71.12"/>
 </segment>
 <segment>
