File: extras/schematic/TFT_ENCODER_CIRCUIT.sch (EAGLE design)
At the start: 18 parts, among them M1 ARDUINO-PRO-MINI-3.3V, U1 SI4703

Commit message: RDA5807 Arduino Library
Parts:
- removed C1, C2: 22pF, capacitor-wima:C2,5-3
- removed C3: 22nF, capacitor-wima:C2,5-3
- removed CX1, CX2: (no value), rcl:CXXC10B6
- removed Q1: (no value), crystal:86SMX
- removed R1, R2: 4.7k, SparkFun-Resistors:4.7KOHM-0603-1/10W-1%
- removed U1: SI4703, SI4703:SI4703
- added ANT1: (no value), discrete:ANTENNA
- added U$1: RDA, RDA:RDA
- J1: device SparkFun-Connectors:AUDIO_JACK_2.5MM_HOLESONLY -> SparkFun-Connectors:AUDIO_JACK_2.5MMSPECIAL_POGO_PINS
Connections:
- removed net N$16: CX1.1, U1.ROUT
- removed net N$19: CX2.1, U1.LOUT
- removed net N$20: CX1.2, J1.RIGHT
- removed net N$21: CX2.2, J1.LEFT
- net GND: now also M1.GND.2, M1.RST.2, U$1.GND; no longer C1.2, C2.2, C3.1, U1.GND@PAD
- net N$1: now also U$1.SCL; no longer R1.1, U1.SCLK
- net N$2: now also U$1.SDA; no longer R2.1, U1.SDIO
- net N$3: now also J1.LEFT, U$1.L; no longer M1.A0, U1.!RST
- net N$4: now also J1.RIGHT, U$1.R; no longer C1.1, Q1.2, U1.GPIO3
- net N$5: now also ANT1.1, U$1.ANT; no longer C2.1, Q1.1, U1.RCLK
- net VCC: now also U$1.VCC; no longer C3.2, R1.2, R2.2, U1.VA, U1.VD
Other:
- note added: "Encoder"
- note added: "RDA5807 module"
- moved on the sheet: J1

Commit message: Extras
Connections:
- removed net N$18: LCD1.CS, M1.D12
- new net N$16: LCD1.CS, M1.D10
- net N$17: now also M1.D12; no longer M1.D10
Changed lines of the file:
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@@
 <drawing>
 <settings>
-<setting alwaysvectorfont="yes"/>
+<setting alwaysvectorfont="no"/>
 <setting verticaltext="up"/>
 </settings>
@@
 <net name="N$17" class="0">
 <segment>
-<pinref part="M1" gate="G$1" pin="D10"/>
-<wire x1="48.26" y1="45.72" x2="55.88" y2="45.72" width="0.1524" layer="91"/>
-<wire x1="55.88" y1="45.72" x2="55.88" y2="7.62" width="0.1524" layer="91"/>
 <wire x1="55.88" y1="7.62" x2="-5.08" y2="7.62" width="0.1524" layer="91"/>
 <pinref part="SEEK" gate="G$1" pin="P$2"/>
 <wire x1="-5.08" y1="7.62" x2="-5.08" y2="22.86" width="0.1524" layer="91"/>
-</segment>
-</net>
-<net name="N$18" class="0">
-<segment>
 <pinref part="M1" gate="G$1" pin="D12"/>
-<wire x1="48.26" y1="50.8" x2="68.58" y2="50.8" width="0.1524" layer="91"/>
-<wire x1="68.58" y1="50.8" x2="68.58" y2="-2.54" width="0.1524" layer="91"/>
-<pinref part="LCD1" gate="G$1" pin="CS"/>
-<wire x1="68.58" y1="-2.54" x2="78.74" y2="-2.54" width="0.1524" layer="91"/>
+<wire x1="48.26" y1="50.8" x2="55.88" y2="50.8" width="0.1524" layer="91"/>
+<wire x1="55.88" y1="50.8" x2="55.88" y2="7.62" width="0.1524" layer="91"/>
 </segment>
 </net>
@@
 </segment>
 </net>
+<net name="N$16" class="0">
+<segment>
+<pinref part="M1" gate="G$1" pin="D10"/>
+<wire x1="48.26" y1="45.72" x2="68.58" y2="45.72" width="0.1524" layer="91"/>
+<pinref part="LCD1" gate="G$1" pin="CS"/>
+<wire x1="68.58" y1="-2.54" x2="78.74" y2="-2.54" width="0.1524" layer="91"/>
+<wire x1="68.58" y1="45.72" x2="68.58" y2="-2.54" width="0.1524" layer="91"/>
+</segment>
+</net>

Commit message: Documentation
Connections:
- net N$17: now also M1.A0; no longer M1.D12
- net VCC: no longer M1.VCC
Other:
- note added: "3.3V"
Changed lines of the file:
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@@
 <text x="99.06" y="86.36" size="1.778" layer="91">RDA5807 module</text>
 <text x="-12.7" y="104.14" size="1.778" layer="91">Encoder</text>
+<text x="78.74" y="68.58" size="1.778" layer="91">3.3V</text>
 </plain>
 <instances>
@@
 <attribute name="VALUE" x="73.66" y="25.4" size="1.778" layer="96" rot="R180"/>
 </instance>
-<instance part="SUPPLY3" gate="G$1" x="48.26" y="2.54" smashed="yes" rot="R90">
-<attribute name="VALUE" x="45.085" y="0.635" size="1.778" layer="96" rot="R90"/>
+<instance part="SUPPLY3" gate="G$1" x="48.26" y="0" smashed="yes" rot="R90">
+<attribute name="VALUE" x="45.085" y="-1.905" size="1.778" layer="96" rot="R90"/>
 </instance>
 <instance part="SUPPLY4" gate="G$1" x="76.2" y="17.78" smashed="yes" rot="R90">
@@
 <net name="VCC" class="0">
 <segment>
-<pinref part="M1" gate="G$1" pin="VCC"/>
 <pinref part="SUPPLY2" gate="G$1" pin="VCC"/>
-<wire x1="48.26" y1="66.04" x2="68.58" y2="66.04" width="0.1524" layer="91"/>
 <pinref part="U$1" gate="G$1" pin="VCC"/>
 <wire x1="95.06" y1="69.82" x2="95.06" y2="66.04" width="0.1524" layer="91"/>
 <wire x1="95.06" y1="66.04" x2="68.58" y2="66.04" width="0.1524" layer="91"/>
-<junction x="68.58" y="66.04"/>
+</segment>
+<segment>
+<pinref part="LCD1" gate="G$1" pin="LEDA"/>
+<pinref part="SUPPLY4" gate="G$1" pin="VCC"/>
+<junction x="78.74" y="17.78"/>
 </segment>
 <segment>
@@
 <pinref part="SUPPLY3" gate="G$1" pin="VCC"/>
 <wire x1="78.74" y1="2.54" x2="50.8" y2="2.54" width="0.1524" layer="91"/>
-</segment>
-<segment>
-<pinref part="LCD1" gate="G$1" pin="LEDA"/>
-<pinref part="SUPPLY4" gate="G$1" pin="VCC"/>
-<junction x="78.74" y="17.78"/>
+<wire x1="50.8" y1="2.54" x2="50.8" y2="0" width="0.1524" layer="91"/>
 </segment>
 </net>
@@
 <net name="N$17" class="0">
 <segment>
-<wire x1="55.88" y1="7.62" x2="-5.08" y2="7.62" width="0.1524" layer="91"/>
 <pinref part="SEEK" gate="G$1" pin="P$2"/>
-<wire x1="-5.08" y1="7.62" x2="-5.08" y2="22.86" width="0.1524" layer="91"/>
-<pinref part="M1" gate="G$1" pin="D12"/>
-<wire x1="48.26" y1="50.8" x2="55.88" y2="50.8" width="0.1524" layer="91"/>
-<wire x1="55.88" y1="50.8" x2="55.88" y2="7.62" width="0.1524" layer="91"/>
-</segment>
-</net>
+<wire x1="-5.08" y1="5.08" x2="-5.08" y2="22.86" width="0.1524" layer="91"/>
+<pinref part="M1" gate="G$1" pin="A0"/>
+<wire x1="48.26" y1="55.88" x2="53.34" y2="55.88" width="0.1524" layer="91"/>
+<wire x1="53.34" y1="55.88" x2="53.34" y2="5.08" width="0.1524" layer="91"/>
+<wire x1="53.34" y1="5.08" x2="-5.08" y2="5.08" width="0.1524" layer="91"/>
+</segment>
+</net>
