File: extras/schematic/basic_circuit.sch (EAGLE design)
At the start: 4 parts, among them M1 ARDUINO-PRO-MINI-3.3V#APC

Commit message: RDA5807 Arduino Library
Parts:
- removed U$2: 1.575GHz, SparkFun-GPS:ANTENNAGPS-2X7MM
- added ANT1: (no value), discrete:ANTENNA
Connections:
- net N$6: now also ANT1.1; no longer U$2.SIGNAL
Changed lines of the file:
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@@
 <part name="GND1" library="supply1" library_urn="urn:adsk.eagle:library:371" deviceset="GND" device=""/>
 <part name="J1" library="SparkFun-Connectors" library_urn="urn:adsk.eagle:library:513" deviceset="AUDIO_JACK_2.5MM" device="SPECIAL_POGO_PINS" package3d_urn="urn:adsk.eagle:package:38005/1"/>
-<part name="U$2" library="SparkFun-GPS" library_urn="urn:adsk.eagle:library:518" deviceset="ANTENNA" device="GPS-2X7MM" package3d_urn="urn:adsk.eagle:package:38594/1" value="1.575GHz"/>
+<part name="ANT1" library="discrete" library_urn="urn:adsk.eagle:library:211" deviceset="ANTENNA" device="" package3d_urn="urn:adsk.eagle:package:12928/1"/>
 </parts>
 <sheets>
@@
 <attribute name="VALUE" x="152.4" y="66.04" size="1.778" layer="96" font="vector" rot="R180"/>
 </instance>
-<instance part="U$2" gate="G$1" x="127" y="88.9" smashed="yes">
-<attribute name="NAME" x="127.508" y="88.9" size="1.778" layer="95" font="vector"/>
-<attribute name="VALUE" x="127.508" y="86.36" size="1.778" layer="96" font="vector"/>
+<instance part="ANT1" gate="A" x="127" y="88.9" smashed="yes">
+<attribute name="NAME" x="124.46" y="90.17" size="1.778" layer="95"/>
+<attribute name="VALUE" x="129.54" y="83.82" size="1.778" layer="96"/>
 </instance>
 </instances>
@@
 <segment>
 <pinref part="U$1" gate="G$1" pin="ANT"/>
-<pinref part="U$2" gate="G$1" pin="SIGNAL"/>
 <wire x1="121.6" y1="69.12" x2="127" y2="69.12" width="0.1524" layer="91"/>
 <wire x1="127" y1="69.12" x2="127" y2="83.82" width="0.1524" layer="91"/>
+<pinref part="ANT1" gate="A" pin="1"/>
+<junction x="127" y="83.82"/>
 </segment>
 </net>

Commit message: Documentation
Connections:
- net VCC: no longer M1.VCC
Other:
- note added: "3.3V"
Changed lines of the file:
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@@
 <drawing>
 <settings>
-<setting alwaysvectorfont="yes"/>
+<setting alwaysvectorfont="no"/>
 <setting verticaltext="up"/>
 </settings>
@@
 <plain>
 <text x="96.52" y="73.66" size="1.778" layer="91">RDA5807 breakout</text>
+<text x="83.82" y="58.42" size="1.778" layer="91">3.3V</text>
 </plain>
 <instances>
@@
 <wire x1="97.6" y1="57.12" x2="97.6" y2="55.88" width="0.1524" layer="91"/>
 <wire x1="97.6" y1="55.88" x2="78.74" y2="55.88" width="0.1524" layer="91"/>
-<pinref part="M1" gate="G$1" pin="VCC"/>
-<wire x1="55.88" y1="63.5" x2="71.12" y2="63.5" width="0.1524" layer="91"/>
-<wire x1="71.12" y1="63.5" x2="71.12" y2="55.88" width="0.1524" layer="91"/>
-<wire x1="71.12" y1="55.88" x2="78.74" y2="55.88" width="0.1524" layer="91"/>
-<junction x="78.74" y="55.88"/>
-</segment>
-</net>
+</segment>
+</net>
