File: extras/schematic/LCD16x02_ENCODER_ESP32_CIRCUIT.sch (EAGLE design)
At the start: 17 parts, among them Q1 32768k, U1 ESP32-DEVKITC-32D, X1 HD44780LCD-1602

Commit message: Documentation
Connections:
- net GND: now also RE1.A
- net N$16: now also RE1.B, U1.IO27; no longer RE1.A
Changed lines of the file:
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@@
 <wire x1="7.62" y1="76.2" x2="7.62" y2="71.12" width="0.1524" layer="91"/>
 <junction x="7.62" y="71.12"/>
+<pinref part="RE1" gate="G$1" pin="A"/>
+<wire x1="7.62" y1="53.34" x2="7.62" y2="71.12" width="0.1524" layer="91"/>
 </segment>
 <segment>
@@
 <pinref part="VR1" gate="G$1" pin="S"/>
 <wire x1="50.8" y1="83.82" x2="12.7" y2="83.82" width="0.1524" layer="91"/>
-</segment>
-</net>
-<net name="N$16" class="0">
-<segment>
-<pinref part="RE1" gate="G$1" pin="A"/>
-<wire x1="7.62" y1="53.34" x2="10.16" y2="53.34" width="0.1524" layer="91"/>
 </segment>
 </net>
@@
 </segment>
 </net>
+<net name="N$16" class="0">
+<segment>
+<pinref part="RE1" gate="G$1" pin="B"/>
+<wire x1="7.62" y1="48.26" x2="12.7" y2="48.26" width="0.1524" layer="91"/>
+<wire x1="12.7" y1="48.26" x2="12.7" y2="-27.94" width="0.1524" layer="91"/>
+<wire x1="12.7" y1="-27.94" x2="58.42" y2="-27.94" width="0.1524" layer="91"/>
+<pinref part="U1" gate="G$1" pin="IO27"/>
+<wire x1="58.42" y1="-27.94" x2="58.42" y2="-12.7" width="0.1524" layer="91"/>
+</segment>
+</net>

Commit message: Documentation
Connections:
- new net N$26: RE1.B, U1.IO14
- new net N$27: RE1.A, U1.IO13
- net GND: no longer RE1.A
- net N$16: now also SEEK.P$2; no longer RE1.B
- net N$21: now also RDS_ON.P$2; no longer SEEK.P$2
Changed lines of the file:
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@@
 <wire x1="7.62" y1="76.2" x2="7.62" y2="71.12" width="0.1524" layer="91"/>
 <junction x="7.62" y="71.12"/>
-<pinref part="RE1" gate="G$1" pin="A"/>
-<wire x1="7.62" y1="53.34" x2="7.62" y2="71.12" width="0.1524" layer="91"/>
 </segment>
 <segment>
@@
 <pinref part="VR1" gate="G$1" pin="S"/>
 <wire x1="50.8" y1="83.82" x2="12.7" y2="83.82" width="0.1524" layer="91"/>
-</segment>
-</net>
-<net name="N$21" class="0">
-<segment>
-<pinref part="SEEK" gate="G$1" pin="P$2"/>
-<wire x1="0" y1="-22.86" x2="0" y2="-15.24" width="0.1524" layer="91"/>
-<pinref part="U1" gate="G$1" pin="IO26"/>
-<wire x1="55.88" y1="-12.7" x2="55.88" y2="-22.86" width="0.1524" layer="91"/>
-<wire x1="55.88" y1="-22.86" x2="0" y2="-22.86" width="0.1524" layer="91"/>
 </segment>
 </net>
@@
 <net name="N$16" class="0">
 <segment>
+<pinref part="SEEK" gate="G$1" pin="P$2"/>
+<wire x1="0" y1="-25.4" x2="0" y2="-15.24" width="0.1524" layer="91"/>
+<pinref part="U1" gate="G$1" pin="IO27"/>
+<wire x1="58.42" y1="-12.7" x2="58.42" y2="-25.4" width="0.1524" layer="91"/>
+<wire x1="58.42" y1="-25.4" x2="0" y2="-25.4" width="0.1524" layer="91"/>
+</segment>
+</net>
+<net name="N$21" class="0">
+<segment>
+<pinref part="RDS_ON" gate="G$1" pin="P$2"/>
+<wire x1="0" y1="-2.54" x2="17.78" y2="-2.54" width="0.1524" layer="91"/>
+<wire x1="17.78" y1="-2.54" x2="17.78" y2="-22.86" width="0.1524" layer="91"/>
+<wire x1="17.78" y1="-22.86" x2="55.88" y2="-22.86" width="0.1524" layer="91"/>
+<pinref part="U1" gate="G$1" pin="IO26"/>
+<wire x1="55.88" y1="-22.86" x2="55.88" y2="-12.7" width="0.1524" layer="91"/>
+</segment>
+</net>
+<net name="N$26" class="0">
+<segment>
 <pinref part="RE1" gate="G$1" pin="B"/>
-<wire x1="7.62" y1="48.26" x2="12.7" y2="48.26" width="0.1524" layer="91"/>
-<wire x1="12.7" y1="48.26" x2="12.7" y2="-27.94" width="0.1524" layer="91"/>
-<wire x1="12.7" y1="-27.94" x2="58.42" y2="-27.94" width="0.1524" layer="91"/>
-<pinref part="U1" gate="G$1" pin="IO27"/>
-<wire x1="58.42" y1="-27.94" x2="58.42" y2="-12.7" width="0.1524" layer="91"/>
-</segment>
-</net>
+<wire x1="7.62" y1="48.26" x2="7.62" y2="-27.94" width="0.1524" layer="91"/>
+<wire x1="7.62" y1="-27.94" x2="60.96" y2="-27.94" width="0.1524" layer="91"/>
+<pinref part="U1" gate="G$1" pin="IO14"/>
+<wire x1="60.96" y1="-27.94" x2="60.96" y2="-12.7" width="0.1524" layer="91"/>
+</segment>
+</net>
+<net name="N$27" class="0">
+<segment>
+<pinref part="RE1" gate="G$1" pin="A"/>
+<wire x1="7.62" y1="53.34" x2="12.7" y2="53.34" width="0.1524" layer="91"/>
+<wire x1="12.7" y1="53.34" x2="12.7" y2="-33.02" width="0.1524" layer="91"/>
+<wire x1="12.7" y1="-33.02" x2="68.58" y2="-33.02" width="0.1524" layer="91"/>
+<wire x1="68.58" y1="-33.02" x2="68.58" y2="-12.7" width="0.1524" layer="91"/>
+<pinref part="U1" gate="G$1" pin="IO13"/>
+</segment>
+</net>

Commit message: Documentation
Connections:
- net N$1: no longer R4.2
- net N$2: no longer R3.2
- net N$4: now also R3.2, R4.2
Other:
- moved on the sheet: R3, R4
Changed lines of the file:
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@@
 <text x="66.04" y="38.1" size="1.778" layer="91">GPIO21 (SDA)</text>
 <text x="66.04" y="33.02" size="1.778" layer="91">GPIO22 (SCLK)</text>
-<text x="114.3" y="-22.86" size="1.778" layer="91">I2C - PULLUP</text>
+<text x="104.14" y="-22.86" size="1.778" layer="91">I2C - PULLUP</text>
 <text x="172.72" y="35.56" size="1.778" layer="91">Audio Amp.</text>
 <text x="22.86" y="58.42" size="1.778" layer="91">GPIO15</text>
@@
 <attribute name="VALUE" x="83.8498" y="-7.6363" size="1.7799" layer="96" rot="R90"/>
 </instance>
-<instance part="R3" gate="G$1" x="106.68" y="-7.62" smashed="yes" rot="R90">
-<attribute name="NAME" x="105.1814" y="-11.43" size="1.778" layer="95" rot="R90"/>
-<attribute name="VALUE" x="109.982" y="-11.43" size="1.778" layer="96" rot="R90"/>
-</instance>
-<instance part="R4" gate="G$1" x="116.84" y="-7.62" smashed="yes" rot="R90">
-<attribute name="NAME" x="115.3414" y="-11.43" size="1.778" layer="95" rot="R90"/>
-<attribute name="VALUE" x="120.142" y="-11.43" size="1.778" layer="96" rot="R90"/>
+<instance part="R3" gate="G$1" x="86.36" y="-20.32" smashed="yes" rot="R90">
+<attribute name="NAME" x="84.8614" y="-24.13" size="1.778" layer="95" rot="R90"/>
+<attribute name="VALUE" x="89.662" y="-24.13" size="1.778" layer="96" rot="R90"/>
+</instance>
+<instance part="R4" gate="G$1" x="96.52" y="-20.32" smashed="yes" rot="R90">
+<attribute name="NAME" x="95.0214" y="-24.13" size="1.778" layer="95" rot="R90"/>
+<attribute name="VALUE" x="99.822" y="-24.13" size="1.778" layer="96" rot="R90"/>
 </instance>
 <instance part="GND1" gate="1" x="111.76" y="38.1" smashed="yes">
@@
 <pinref part="U$1" gate="G$1" pin="SCLK"/>
 <wire x1="114.3" y1="17.78" x2="116.84" y2="17.78" width="0.1524" layer="91"/>
-<pinref part="R4" gate="G$1" pin="2"/>
-<wire x1="116.84" y1="-2.54" x2="116.84" y2="17.78" width="0.1524" layer="91"/>
-<junction x="116.84" y="17.78"/>
 </segment>
 </net>
@@
 <pinref part="U$1" gate="G$1" pin="SDA"/>
 <wire x1="106.68" y1="12.7" x2="116.84" y2="12.7" width="0.1524" layer="91"/>
-<pinref part="R3" gate="G$1" pin="2"/>
-<wire x1="106.68" y1="-2.54" x2="106.68" y2="12.7" width="0.1524" layer="91"/>
-<junction x="106.68" y="12.7"/>
 </segment>
 </net>
@@
 <pinref part="U1" gate="G$1" pin="IO21"/>
 <wire x1="45.72" y1="27.94" x2="45.72" y2="38.1" width="0.1524" layer="91"/>
-<wire x1="45.72" y1="38.1" x2="96.52" y2="38.1" width="0.1524" layer="91"/>
+<wire x1="45.72" y1="38.1" x2="88.9" y2="38.1" width="0.1524" layer="91"/>
 <pinref part="R2" gate="G$1" pin="1"/>
+<wire x1="88.9" y1="38.1" x2="96.52" y2="38.1" width="0.1524" layer="91"/>
 <wire x1="96.52" y1="38.1" x2="96.52" y2="12.7" width="0.1524" layer="91"/>
+<pinref part="R3" gate="G$1" pin="2"/>
+<wire x1="86.36" y1="-15.24" x2="88.9" y2="-15.24" width="0.1524" layer="91"/>
+<wire x1="88.9" y1="-15.24" x2="88.9" y2="38.1" width="0.1524" layer="91"/>
+<junction x="88.9" y="38.1"/>
+<pinref part="R4" gate="G$1" pin="2"/>
+<wire x1="96.52" y1="-15.24" x2="96.52" y2="12.7" width="0.1524" layer="91"/>
+<junction x="96.52" y="12.7"/>
 </segment>
 </net>
@@
 <pinref part="U1" gate="G$1" pin="IO22"/>
 <wire x1="38.1" y1="27.94" x2="38.1" y2="33.02" width="0.1524" layer="91"/>
-</segment>
-</net>
-<net name="N$6" class="0">
-<segment>
-<pinref part="R3" gate="G$1" pin="1"/>
-<pinref part="R4" gate="G$1" pin="1"/>
-<wire x1="106.68" y1="-12.7" x2="111.76" y2="-12.7" width="0.1524" layer="91"/>
-<pinref part="U1" gate="G$1" pin="3V3"/>
-<wire x1="111.76" y1="-12.7" x2="116.84" y2="-12.7" width="0.1524" layer="91"/>
-<wire x1="33.02" y1="-12.7" x2="33.02" y2="-30.48" width="0.1524" layer="91"/>
-<wire x1="33.02" y1="-30.48" x2="111.76" y2="-30.48" width="0.1524" layer="91"/>
-<wire x1="111.76" y1="-30.48" x2="180.34" y2="-30.48" width="0.1524" layer="91"/>
-<wire x1="180.34" y1="-30.48" x2="180.34" y2="17.78" width="0.1524" layer="91"/>
-<pinref part="U$1" gate="G$1" pin="VDD"/>
-<wire x1="180.34" y1="17.78" x2="152.4" y2="17.78" width="0.1524" layer="91"/>
-<wire x1="111.76" y1="-12.7" x2="111.76" y2="-30.48" width="0.1524" layer="91"/>
-<junction x="111.76" y="-12.7"/>
-<junction x="111.76" y="-30.48"/>
 </segment>
 </net>
@@
 </segment>
 </net>
+<net name="N$25" class="0">
+<segment>
+<pinref part="R4" gate="G$1" pin="1"/>
+<pinref part="R3" gate="G$1" pin="1"/>
+<wire x1="86.36" y1="-25.4" x2="91.44" y2="-25.4" width="0.1524" layer="91"/>
+<pinref part="U1" gate="G$1" pin="3V3"/>
+<wire x1="91.44" y1="-25.4" x2="96.52" y2="-25.4" width="0.1524" layer="91"/>
+<wire x1="33.02" y1="-12.7" x2="33.02" y2="-30.48" width="0.1524" layer="91"/>
+<wire x1="33.02" y1="-30.48" x2="91.44" y2="-30.48" width="0.1524" layer="91"/>
+<wire x1="91.44" y1="-30.48" x2="172.72" y2="-30.48" width="0.1524" layer="91"/>
+<wire x1="91.44" y1="-25.4" x2="91.44" y2="-30.48" width="0.1524" layer="91"/>
+<junction x="91.44" y="-25.4"/>
+<junction x="91.44" y="-30.48"/>
+<pinref part="U$1" gate="G$1" pin="VDD"/>
+<wire x1="152.4" y1="17.78" x2="172.72" y2="17.78" width="0.1524" layer="91"/>
+<wire x1="172.72" y1="17.78" x2="172.72" y2="-30.48" width="0.1524" layer="91"/>
+</segment>
+</net>

Commit message: Documentation
Connections:
- net N$4: no longer R3.2
- net N$5: now also R3.2
Changed lines of the file:
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@@
 <pinref part="U1" gate="G$1" pin="IO21"/>
 <wire x1="45.72" y1="27.94" x2="45.72" y2="38.1" width="0.1524" layer="91"/>
-<wire x1="45.72" y1="38.1" x2="88.9" y2="38.1" width="0.1524" layer="91"/>
+<wire x1="45.72" y1="38.1" x2="96.52" y2="38.1" width="0.1524" layer="91"/>
 <pinref part="R2" gate="G$1" pin="1"/>
-<wire x1="88.9" y1="38.1" x2="96.52" y2="38.1" width="0.1524" layer="91"/>
 <wire x1="96.52" y1="38.1" x2="96.52" y2="12.7" width="0.1524" layer="91"/>
-<pinref part="R3" gate="G$1" pin="2"/>
-<wire x1="86.36" y1="-15.24" x2="88.9" y2="-15.24" width="0.1524" layer="91"/>
-<wire x1="88.9" y1="-15.24" x2="88.9" y2="38.1" width="0.1524" layer="91"/>
-<junction x="88.9" y="38.1"/>
 <pinref part="R4" gate="G$1" pin="2"/>
 <wire x1="96.52" y1="-15.24" x2="96.52" y2="12.7" width="0.1524" layer="91"/>
@@
 <segment>
 <pinref part="R1" gate="G$1" pin="1"/>
-<wire x1="38.1" y1="33.02" x2="104.14" y2="33.02" width="0.1524" layer="91"/>
+<wire x1="38.1" y1="33.02" x2="86.36" y2="33.02" width="0.1524" layer="91"/>
+<wire x1="86.36" y1="33.02" x2="104.14" y2="33.02" width="0.1524" layer="91"/>
 <wire x1="104.14" y1="33.02" x2="104.14" y2="17.78" width="0.1524" layer="91"/>
 <pinref part="U1" gate="G$1" pin="IO22"/>
 <wire x1="38.1" y1="27.94" x2="38.1" y2="33.02" width="0.1524" layer="91"/>
+<pinref part="R3" gate="G$1" pin="2"/>
+<wire x1="86.36" y1="-15.24" x2="86.36" y2="33.02" width="0.1524" layer="91"/>
+<junction x="86.36" y="33.02"/>
 </segment>
 </net>
