File: extras/schematic/minimalist_receiver_circuit.sch (EAGLE design)
At the start: 6 parts, among them M1 ARDUINO-PRO-MINI-3.3V#APC

Commit message: Documentation
Parts:
- renumbered SEEKDOWN1 to SEEK_DOWN, SEEKDUP to SEEKD_UP
Changed lines of the file:
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@@
 <part name="ANT1" library="discrete" library_urn="urn:adsk.eagle:library:211" deviceset="ANTENNA" device="" package3d_urn="urn:adsk.eagle:package:12928/1"/>
 <part name="GND2" library="supply1" library_urn="urn:adsk.eagle:library:371" deviceset="GND" device=""/>
-<part name="SEEKDUP" library="SparkFun-Switches" deviceset="MOMENTARY-SWITCH-SPST" device="-PTH-6.0MM"/>
-<part name="SEEKDOWN1" library="SparkFun-Switches" deviceset="MOMENTARY-SWITCH-SPST" device="-PTH-6.0MM"/>
+<part name="SEEKD_UP" library="SparkFun-Switches" deviceset="MOMENTARY-SWITCH-SPST" device="-PTH-6.0MM"/>
+<part name="SEEK_DOWN" library="SparkFun-Switches" deviceset="MOMENTARY-SWITCH-SPST" device="-PTH-6.0MM"/>
 <part name="GND3" library="supply1" library_urn="urn:adsk.eagle:library:371" deviceset="GND" device=""/>
 <part name="SUPPLY2" library="supply2" library_urn="urn:adsk.eagle:library:372" deviceset="VCC" device=""/>
@@
 <attribute name="VALUE" x="76.2" y="22.86" size="1.778" layer="96"/>
 </instance>
-<instance part="SEEKDUP" gate="G$1" x="12.7" y="55.88" smashed="yes">
+<instance part="SEEKD_UP" gate="G$1" x="12.7" y="55.88" smashed="yes">
 <attribute name="NAME" x="12.7" y="57.404" size="1.778" layer="95" font="vector" align="bottom-center"/>
 </instance>
-<instance part="SEEKDOWN1" gate="G$1" x="12.7" y="48.26" smashed="yes">
+<instance part="SEEK_DOWN" gate="G$1" x="12.7" y="48.26" smashed="yes">
 <attribute name="NAME" x="12.7" y="49.784" size="1.778" layer="95" font="vector" align="bottom-center"/>
 </instance>
@@
 </segment>
 <segment>
-<pinref part="SEEKDUP" gate="G$1" pin="1"/>
+<pinref part="SEEKD_UP" gate="G$1" pin="1"/>
 <wire x1="7.62" y1="55.88" x2="2.54" y2="55.88" width="0.1524" layer="91"/>
 <pinref part="GND3" gate="1" pin="GND"/>
 <wire x1="2.54" y1="55.88" x2="2.54" y2="48.26" width="0.1524" layer="91"/>
-<pinref part="SEEKDOWN1" gate="G$1" pin="1"/>
+<pinref part="SEEK_DOWN" gate="G$1" pin="1"/>
 <wire x1="2.54" y1="48.26" x2="2.54" y2="38.1" width="0.1524" layer="91"/>
 <wire x1="7.62" y1="48.26" x2="2.54" y2="48.26" width="0.1524" layer="91"/>
@@
 <net name="N$7" class="0">
 <segment>
-<pinref part="SEEKDUP" gate="G$1" pin="2"/>
+<pinref part="SEEKD_UP" gate="G$1" pin="2"/>
 <pinref part="M1" gate="G$1" pin="D4"/>
 <wire x1="17.78" y1="55.88" x2="40.64" y2="55.88" width="0.1524" layer="91"/>
@@
 <net name="N$8" class="0">
 <segment>
-<pinref part="SEEKDOWN1" gate="G$1" pin="2"/>
+<pinref part="SEEK_DOWN" gate="G$1" pin="2"/>
 <wire x1="17.78" y1="48.26" x2="25.4" y2="48.26" width="0.1524" layer="91"/>
 <wire x1="25.4" y1="48.26" x2="25.4" y2="53.34" width="0.1524" layer="91"/>

Commit message: Extras
Other:
- note added: "ATmega328 Based Board"
- note added: "Arduino"
- note removed: "Atmega Based Board"
Changed lines of the file:
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@@
 <text x="109.22" y="73.66" size="1.778" layer="91">RDA5807 breakout</text>
 <text x="96.52" y="58.42" size="1.778" layer="91">3.3V</text>
-<text x="48.26" y="91.44" size="1.778" layer="91">Atmega Based Board</text>
+<text x="45.72" y="91.44" size="1.778" layer="91">ATmega328 Based Board</text>
 <text x="71.12" y="106.68" size="1.778" layer="91">Minimalist Receiver based on RDA5807</text>
+<text x="53.34" y="93.98" size="1.778" layer="91">Arduino</text>
 </plain>
 <instances>

Commit message: Extras
Parts:
- renumbered SEEKD_UP to SEEKD_DOWN, SEEK_DOWN to SEEK_UP
Changed lines of the file:
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@@
 <part name="ANT1" library="discrete" library_urn="urn:adsk.eagle:library:211" deviceset="ANTENNA" device="" package3d_urn="urn:adsk.eagle:package:12928/1"/>
 <part name="GND2" library="supply1" library_urn="urn:adsk.eagle:library:371" deviceset="GND" device=""/>
-<part name="SEEKD_UP" library="SparkFun-Switches" deviceset="MOMENTARY-SWITCH-SPST" device="-PTH-6.0MM"/>
-<part name="SEEK_DOWN" library="SparkFun-Switches" deviceset="MOMENTARY-SWITCH-SPST" device="-PTH-6.0MM"/>
+<part name="SEEKD_DOWN" library="SparkFun-Switches" deviceset="MOMENTARY-SWITCH-SPST" device="-PTH-6.0MM"/>
+<part name="SEEK_UP" library="SparkFun-Switches" deviceset="MOMENTARY-SWITCH-SPST" device="-PTH-6.0MM"/>
 <part name="GND3" library="supply1" library_urn="urn:adsk.eagle:library:371" deviceset="GND" device=""/>
 <part name="SUPPLY2" library="supply2" library_urn="urn:adsk.eagle:library:372" deviceset="VCC" device=""/>
@@
 <attribute name="VALUE" x="76.2" y="22.86" size="1.778" layer="96"/>
 </instance>
-<instance part="SEEKD_UP" gate="G$1" x="12.7" y="55.88" smashed="yes">
+<instance part="SEEKD_DOWN" gate="G$1" x="12.7" y="55.88" smashed="yes">
 <attribute name="NAME" x="12.7" y="57.404" size="1.778" layer="95" font="vector" align="bottom-center"/>
 </instance>
-<instance part="SEEK_DOWN" gate="G$1" x="12.7" y="48.26" smashed="yes">
+<instance part="SEEK_UP" gate="G$1" x="12.7" y="48.26" smashed="yes">
 <attribute name="NAME" x="12.7" y="49.784" size="1.778" layer="95" font="vector" align="bottom-center"/>
 </instance>
@@
 </segment>
 <segment>
-<pinref part="SEEKD_UP" gate="G$1" pin="1"/>
+<pinref part="SEEKD_DOWN" gate="G$1" pin="1"/>
 <wire x1="7.62" y1="55.88" x2="2.54" y2="55.88" width="0.1524" layer="91"/>
 <pinref part="GND3" gate="1" pin="GND"/>
 <wire x1="2.54" y1="55.88" x2="2.54" y2="48.26" width="0.1524" layer="91"/>
-<pinref part="SEEK_DOWN" gate="G$1" pin="1"/>
+<pinref part="SEEK_UP" gate="G$1" pin="1"/>
 <wire x1="2.54" y1="48.26" x2="2.54" y2="38.1" width="0.1524" layer="91"/>
 <wire x1="7.62" y1="48.26" x2="2.54" y2="48.26" width="0.1524" layer="91"/>
@@
 <net name="N$7" class="0">
 <segment>
-<pinref part="SEEKD_UP" gate="G$1" pin="2"/>
+<pinref part="SEEKD_DOWN" gate="G$1" pin="2"/>
 <pinref part="M1" gate="G$1" pin="D4"/>
 <wire x1="17.78" y1="55.88" x2="40.64" y2="55.88" width="0.1524" layer="91"/>
@@
 <net name="N$8" class="0">
 <segment>
-<pinref part="SEEK_DOWN" gate="G$1" pin="2"/>
+<pinref part="SEEK_UP" gate="G$1" pin="2"/>
 <wire x1="17.78" y1="48.26" x2="25.4" y2="48.26" width="0.1524" layer="91"/>
 <wire x1="25.4" y1="48.26" x2="25.4" y2="53.34" width="0.1524" layer="91"/>

Commit message: Extras
Parts:
- renumbered SEEKD_DOWN to SEEK_DOWN
Changed lines of the file:
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@@
 <part name="ANT1" library="discrete" library_urn="urn:adsk.eagle:library:211" deviceset="ANTENNA" device="" package3d_urn="urn:adsk.eagle:package:12928/1"/>
 <part name="GND2" library="supply1" library_urn="urn:adsk.eagle:library:371" deviceset="GND" device=""/>
-<part name="SEEKD_DOWN" library="SparkFun-Switches" deviceset="MOMENTARY-SWITCH-SPST" device="-PTH-6.0MM"/>
+<part name="SEEK_DOWN" library="SparkFun-Switches" deviceset="MOMENTARY-SWITCH-SPST" device="-PTH-6.0MM"/>
 <part name="SEEK_UP" library="SparkFun-Switches" deviceset="MOMENTARY-SWITCH-SPST" device="-PTH-6.0MM"/>
 <part name="GND3" library="supply1" library_urn="urn:adsk.eagle:library:371" deviceset="GND" device=""/>
@@
 <attribute name="VALUE" x="76.2" y="22.86" size="1.778" layer="96"/>
 </instance>
-<instance part="SEEKD_DOWN" gate="G$1" x="12.7" y="55.88" smashed="yes">
+<instance part="SEEK_DOWN" gate="G$1" x="12.7" y="55.88" smashed="yes">
 <attribute name="NAME" x="12.7" y="57.404" size="1.778" layer="95" font="vector" align="bottom-center"/>
 </instance>
@@
 </segment>
 <segment>
-<pinref part="SEEKD_DOWN" gate="G$1" pin="1"/>
+<pinref part="SEEK_DOWN" gate="G$1" pin="1"/>
 <wire x1="7.62" y1="55.88" x2="2.54" y2="55.88" width="0.1524" layer="91"/>
 <pinref part="GND3" gate="1" pin="GND"/>
@@
 <net name="N$7" class="0">
 <segment>
-<pinref part="SEEKD_DOWN" gate="G$1" pin="2"/>
+<pinref part="SEEK_DOWN" gate="G$1" pin="2"/>
 <pinref part="M1" gate="G$1" pin="D4"/>
 <wire x1="17.78" y1="55.88" x2="40.64" y2="55.88" width="0.1524" layer="91"/>
