File: extras/schematic/basic_attiny84.sch (EAGLE design)
At the start: 14 parts, among them U1 SI4703

Commit message: Extras
Parts:
- removed C1, C2: 22pF, capacitor-wima:C2,5-3
- removed C3: 22nF, capacitor-wima:C2,5-3
- removed CX1, CX2: (no value), rcl:CXXC10B6
- removed Q1: (no value), crystal:86SMX
- removed R1, R2: 4.7k, SparkFun-Resistors:4.7KOHM-0603-1/10W-1%
- removed U1: SI4703, SI4703:SI4703
- added ANT1: (no value), discrete:ANTENNA
- added U$2: RDA, RDA:RDA
- J1: device SparkFun-Connectors:AUDIO_JACK_2.5MM_HOLESONLY -> SparkFun-Connectors:AUDIO_JACK_2.5MMSPECIAL_POGO_PINS
Connections:
- removed net N$16: CX1.1, U1.ROUT
- removed net N$19: CX2.1, U1.LOUT
- removed net N$20: CX1.2, J1.RIGHT
- removed net N$21: CX2.2, J1.LEFT
- net GND: now also U$2.GND; no longer C1.2, C2.2, C3.1, U1.GND@PAD
- net N$1: now also U$1.(PCINT6/OC1A/SDA/MOSI/ADC6)PA6, U$2.SDA; no longer R1.1, U$1.(PCINT4/T1/SCL/USCK/ADC4)PA4, U1.SCLK
- net N$2: now also U$1.(PCINT4/T1/SCL/USCK/ADC4)PA4, U$2.SCL; no longer R2.1, U$1.(PCINT6/OC1A/SDA/MOSI/ADC6)PA6, U1.SDIO
- net N$3: now also J1.LEFT, U$2.L; no longer U$1.(PCINT7/ICP/OC0B/ADC7)PA7, U1.!RST
- net N$4: now also J1.RIGHT, U$2.R; no longer C1.1, Q1.2, U1.GPIO3
- net N$5: now also ANT1.1, U$2.ANT; no longer C2.1, Q1.1, U1.RCLK
- net VCC: now also U$2.VCC; no longer C3.2, R1.2, R2.2, U1.VA, U1.VD
Other:
- moved on the sheet: J1

Commit message: RDA5807 Arduino Library
Other:
- note added: "Encoder"
- note added: "RDA5807"
Changed lines of the file:
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@@
 <sheet>
 <plain>
+<text x="58.42" y="96.52" size="1.778" layer="91">RDA5807</text>
+<text x="12.7" y="48.26" size="1.778" layer="91">Encoder</text>
 </plain>
 <instances>

Commit message: RDA5807 Arduino Library
Parts:
- added U$3: DISPLAY-OLED-128X64-I2C, diy-modules:DISPLAY-OLED-128X64-I2C
Connections:
- net GND: now also U$3.GND
- net N$1: now also U$3.SDA
- net N$8: now also U$3.SCL
- net VCC: now also U$3.VCC
Changed lines of the file:
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@@
 <drawing>
 <settings>
-<setting alwaysvectorfont="yes"/>
+<setting alwaysvectorfont="no"/>
 <setting verticaltext="up"/>
 </settings>
@@
 <part name="ANT1" library="discrete" library_urn="urn:adsk.eagle:library:211" deviceset="ANTENNA" device="" package3d_urn="urn:adsk.eagle:package:12928/1"/>
 <part name="SUPPLY1" library="supply2" library_urn="urn:adsk.eagle:library:372" deviceset="VCC" device=""/>
+<part name="U$3" library="diy-modules" deviceset="DISPLAY-OLED-128X64-I2C" device=""/>
+<part name="SUPPLY3" library="supply2" library_urn="urn:adsk.eagle:library:372" deviceset="VCC" device=""/>
+<part name="GND3" library="supply1" library_urn="urn:adsk.eagle:library:371" deviceset="GND" device=""/>
 </parts>
 <sheets>
@@
 <attribute name="VALUE" x="43.815" y="84.455" size="1.778" layer="96"/>
 </instance>
+<instance part="U$3" gate="G$1" x="17.78" y="111.76" smashed="yes" rot="R180"/>
+<instance part="SUPPLY3" gate="G$1" x="20.32" y="78.74" smashed="yes" rot="R180">
+<attribute name="VALUE" x="24.765" y="75.565" size="1.778" layer="96" rot="R180"/>
+</instance>
+<instance part="GND3" gate="1" x="30.48" y="76.2" smashed="yes">
+<attribute name="VALUE" x="27.94" y="73.66" size="1.778" layer="96"/>
+</instance>
 </instances>
 <busses>
@@
 <wire x1="86.36" y1="79.98" x2="86.36" y2="71.12" width="0.1524" layer="91"/>
 </segment>
+<segment>
+<pinref part="GND3" gate="1" pin="GND"/>
+<wire x1="30.48" y1="78.74" x2="22.86" y2="78.74" width="0.1524" layer="91"/>
+<pinref part="U$3" gate="G$1" pin="GND"/>
+<wire x1="22.86" y1="78.74" x2="22.86" y2="91.44" width="0.1524" layer="91"/>
+</segment>
 </net>
 <net name="VCC" class="0">
@@
 <wire x1="53.34" y1="79.98" x2="51.88" y2="79.98" width="0.1524" layer="91"/>
 </segment>
+<segment>
+<pinref part="SUPPLY3" gate="G$1" pin="VCC"/>
+<pinref part="U$3" gate="G$1" pin="VCC"/>
+<wire x1="20.32" y1="81.28" x2="20.32" y2="91.44" width="0.1524" layer="91"/>
+</segment>
 </net>
 <net name="N$6" class="0">
@@
 <pinref part="SEEK_DOWN" gate="G$1" pin="P$1"/>
 <pinref part="U$1" gate="G$1" pin="(PCINT5/OC1B/MISO/DO/ADC5)PA5"/>
-<wire x1="0" y1="68.58" x2="50.8" y2="68.58" width="0.1524" layer="91"/>
+<wire x1="0" y1="68.58" x2="17.78" y2="68.58" width="0.1524" layer="91"/>
+<wire x1="17.78" y1="68.58" x2="50.8" y2="68.58" width="0.1524" layer="91"/>
 <wire x1="50.8" y1="68.58" x2="50.8" y2="45.72" width="0.1524" layer="91"/>
+<pinref part="U$3" gate="G$1" pin="SCL"/>
+<wire x1="17.78" y1="91.44" x2="17.78" y2="68.58" width="0.1524" layer="91"/>
+<junction x="17.78" y="68.58"/>
 </segment>
 </net>
@@
 <wire x1="35.56" y1="91.98" x2="35.56" y2="71.12" width="0.1524" layer="91"/>
 <pinref part="U$1" gate="G$1" pin="(PCINT6/OC1A/SDA/MOSI/ADC6)PA6"/>
-<wire x1="35.56" y1="71.12" x2="0" y2="71.12" width="0.1524" layer="91"/>
-</segment>
-</net>
+<wire x1="35.56" y1="71.12" x2="15.24" y2="71.12" width="0.1524" layer="91"/>
+<pinref part="U$3" gate="G$1" pin="SDA"/>
+<wire x1="15.24" y1="71.12" x2="0" y2="71.12" width="0.1524" layer="91"/>
+<wire x1="15.24" y1="91.44" x2="15.24" y2="71.12" width="0.1524" layer="91"/>
+<junction x="15.24" y="71.12"/>
+</segment>
+</net>
