File: extras/schematic/basic_attiny85.sch (EAGLE design)
At the start: 10 parts, among them U2 ATTINY85-20P

Commit message: RDA5807 Arduino Library
Parts:
- removed R1, R2: 4.7k, SparkFun-Resistors:4.7KOHM-0603-1/10W-1%
- added U$2: DISPLAY-OLED-128X64-I2C, diy-modules:DISPLAY-OLED-128X64-I2C
Connections:
- removed net N$3: U$1.SDA, U2.PB3
- net GND: now also U$2.GND
- net N$1: now also U$1.SDA, U$2.SDA, U2.PB0; no longer R1.1, U$1.SCL, U2.PB2
- net N$2: now also U$1.SCL, U$2.SCL, U2.PB2; no longer R2.1, U2.PB0
- net VCC: now also U$2.VCC; no longer R1.2, R2.2
Other:
- note added: "SCL"
- note added: "SDA"
Changed lines of the file:
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@@
 <part name="GND2" library="supply1" library_urn="urn:adsk.eagle:library:371" deviceset="GND" device=""/>
 <part name="SUPPLY2" library="supply2" library_urn="urn:adsk.eagle:library:372" deviceset="VCC" device=""/>
-<part name="R1" library="SparkFun-Resistors" library_urn="urn:adsk.eagle:library:532" deviceset="4.7KOHM" device="-0603-1/10W-1%" package3d_urn="urn:adsk.eagle:package:39650/1" value="4.7k"/>
-<part name="R2" library="SparkFun-Resistors" library_urn="urn:adsk.eagle:library:532" deviceset="4.7KOHM" device="-0603-1/10W-1%" package3d_urn="urn:adsk.eagle:package:39650/1" value="4.7k"/>
-<part name="SUPPLY5" library="supply2" library_urn="urn:adsk.eagle:library:372" deviceset="VCC" device=""/>
 <part name="J1" library="SparkFun-Connectors" library_urn="urn:adsk.eagle:library:513" deviceset="AUDIO_JACK_2.5MM" device="_HOLESONLY" package3d_urn="urn:adsk.eagle:package:37993/1"/>
 <part name="CX1" library="rcl" library_urn="urn:adsk.eagle:library:334" deviceset="CX" device="XC10B6" package3d_urn="urn:adsk.eagle:package:23700/1" value="4.7uF"/>
@@
 <attribute name="C" value="1nF"/>
 </part>
+<part name="U$2" library="diy-modules" deviceset="DISPLAY-OLED-128X64-I2C" device=""/>
+<part name="SUPPLY3" library="supply2" library_urn="urn:adsk.eagle:library:372" deviceset="VCC" device=""/>
+<part name="GND3" library="supply1" library_urn="urn:adsk.eagle:library:371" deviceset="GND" device=""/>
 </parts>
 <sheets>
 <sheet>
 <plain>
+<text x="35.56" y="71.12" size="1.778" layer="91">SCL</text>
+<text x="35.56" y="66.04" size="1.778" layer="91">SDA</text>
 </plain>
 <instances>
@@
 <attribute name="VALUE" x="-6.985" y="92.075" size="1.778" layer="96"/>
 </instance>
-<instance part="R1" gate="G$1" x="50.8" y="93.98" smashed="yes" rot="R90">
-<attribute name="NAME" x="49.276" y="93.98" size="1.778" layer="95" font="vector" rot="R90" align="bottom-center"/>
-<attribute name="VALUE" x="52.324" y="93.98" size="1.778" layer="96" font="vector" rot="R90" align="top-center"/>
-</instance>
-<instance part="R2" gate="G$1" x="58.42" y="93.98" smashed="yes" rot="R90">
-<attribute name="NAME" x="56.896" y="93.98" size="1.778" layer="95" font="vector" rot="R90" align="bottom-center"/>
-<attribute name="VALUE" x="59.944" y="93.98" size="1.778" layer="96" font="vector" rot="R90" align="top-center"/>
-</instance>
-<instance part="SUPPLY5" gate="G$1" x="53.34" y="101.6" smashed="yes">
-<attribute name="VALUE" x="51.435" y="104.775" size="1.778" layer="96"/>
-</instance>
 <instance part="J1" gate="G$1" x="124.46" y="38.1" smashed="yes" rot="R90">
 <attribute name="NAME" x="121.412" y="33.02" size="1.778" layer="95" font="vector" rot="R90"/>
@@
 <instance part="C1" gate="G$1" x="106.68" y="88.9" smashed="yes">
 <attribute name="C" x="106.68" y="88.9" size="1.778" layer="96"/>
+</instance>
+<instance part="U$2" gate="G$1" x="55.88" y="106.68" smashed="yes" rot="R180">
+<attribute name="NAME" x="40.64" y="93.98" size="1.778" layer="95" rot="R180"/>
+<attribute name="VALUE" x="40.64" y="96.52" size="1.778" layer="96" rot="R180"/>
+</instance>
+<instance part="SUPPLY3" gate="G$1" x="58.42" y="78.74" smashed="yes" rot="R180">
+<attribute name="VALUE" x="62.865" y="75.565" size="1.778" layer="96" rot="R180"/>
+</instance>
+<instance part="GND3" gate="1" x="66.04" y="83.82" smashed="yes">
+<attribute name="VALUE" x="63.5" y="81.28" size="1.778" layer="96"/>
 </instance>
 </instances>
@@
 </busses>
 <nets>
-<net name="N$1" class="0">
-<segment>
-<pinref part="R1" gate="G$1" pin="1"/>
-<pinref part="U2" gate="G$1" pin="PB2"/>
-<wire x1="35.56" y1="71.12" x2="50.8" y2="71.12" width="0.1524" layer="91"/>
-<wire x1="50.8" y1="71.12" x2="50.8" y2="88.9" width="0.1524" layer="91"/>
-<pinref part="U$1" gate="G$1" pin="SCL"/>
-<wire x1="79.82" y1="68.66" x2="63.5" y2="68.66" width="0.1524" layer="91"/>
-<wire x1="63.5" y1="68.66" x2="63.5" y2="71.12" width="0.1524" layer="91"/>
-<wire x1="63.5" y1="71.12" x2="50.8" y2="71.12" width="0.1524" layer="91"/>
-<junction x="50.8" y="71.12"/>
-</segment>
-</net>
-<net name="N$2" class="0">
-<segment>
-<pinref part="R2" gate="G$1" pin="1"/>
-<pinref part="U2" gate="G$1" pin="PB0"/>
-<wire x1="58.42" y1="88.9" x2="58.42" y2="66.04" width="0.1524" layer="91"/>
-<wire x1="58.42" y1="66.04" x2="35.56" y2="66.04" width="0.1524" layer="91"/>
-</segment>
-</net>
 <net name="GND" class="0">
 <segment>
@@
 <junction x="45.72" y="35.56"/>
 </segment>
+<segment>
+<pinref part="U$2" gate="G$1" pin="GND"/>
+<pinref part="GND3" gate="1" pin="GND"/>
+<wire x1="60.96" y1="86.36" x2="66.04" y2="86.36" width="0.1524" layer="91"/>
+</segment>
 </net>
 <net name="VCC" class="0">
-<segment>
-<pinref part="R1" gate="G$1" pin="2"/>
-<pinref part="R2" gate="G$1" pin="2"/>
-<wire x1="50.8" y1="99.06" x2="53.34" y2="99.06" width="0.1524" layer="91"/>
-<pinref part="SUPPLY5" gate="G$1" pin="VCC"/>
-<wire x1="53.34" y1="99.06" x2="58.42" y2="99.06" width="0.1524" layer="91"/>
-<junction x="53.34" y="99.06"/>
-</segment>
 <segment>
 <pinref part="SUPPLY2" gate="G$1" pin="VCC"/>
@@
 <wire x1="79.82" y1="55.88" x2="76.2" y2="55.88" width="0.1524" layer="91"/>
 </segment>
+<segment>
+<pinref part="U$2" gate="G$1" pin="VCC"/>
+<pinref part="SUPPLY3" gate="G$1" pin="VCC"/>
+<wire x1="58.42" y1="86.36" x2="58.42" y2="81.28" width="0.1524" layer="91"/>
+</segment>
 </net>
 <net name="N$16" class="0">
@@
 <wire x1="127" y1="43.18" x2="127" y2="48.26" width="0.1524" layer="91"/>
 <wire x1="127" y1="48.26" x2="129.54" y2="48.26" width="0.1524" layer="91"/>
-</segment>
-</net>
-<net name="N$3" class="0">
-<segment>
-<pinref part="U2" gate="G$1" pin="PB3"/>
-<wire x1="66.04" y1="73.66" x2="35.56" y2="73.66" width="0.1524" layer="91"/>
-<pinref part="U$1" gate="G$1" pin="SDA"/>
-<wire x1="79.82" y1="71.66" x2="66.04" y2="71.66" width="0.1524" layer="91"/>
-<wire x1="66.04" y1="71.66" x2="66.04" y2="73.66" width="0.1524" layer="91"/>
 </segment>
 </net>
@@
 </segment>
 </net>
+<net name="N$1" class="0">
+<segment>
+<pinref part="U2" gate="G$1" pin="PB0"/>
+<wire x1="35.56" y1="66.04" x2="53.34" y2="66.04" width="0.1524" layer="91"/>
+<pinref part="U$1" gate="G$1" pin="SDA"/>
+<wire x1="53.34" y1="66.04" x2="63.5" y2="66.04" width="0.1524" layer="91"/>
+<wire x1="79.82" y1="71.66" x2="63.5" y2="71.66" width="0.1524" layer="91"/>
+<wire x1="63.5" y1="71.66" x2="63.5" y2="66.04" width="0.1524" layer="91"/>
+<pinref part="U$2" gate="G$1" pin="SDA"/>
+<wire x1="53.34" y1="86.36" x2="53.34" y2="66.04" width="0.1524" layer="91"/>
+<junction x="53.34" y="66.04"/>
+</segment>
+</net>
+<net name="N$2" class="0">
+<segment>
+<pinref part="U2" gate="G$1" pin="PB2"/>
+<wire x1="35.56" y1="71.12" x2="55.88" y2="71.12" width="0.1524" layer="91"/>
+<wire x1="55.88" y1="71.12" x2="60.96" y2="71.12" width="0.1524" layer="91"/>
+<wire x1="60.96" y1="71.12" x2="60.96" y2="68.58" width="0.1524" layer="91"/>
+<pinref part="U$1" gate="G$1" pin="SCL"/>
+<wire x1="60.96" y1="68.58" x2="79.82" y2="68.58" width="0.1524" layer="91"/>
+<wire x1="79.82" y1="68.58" x2="79.82" y2="68.66" width="0.1524" layer="91"/>
+<pinref part="U$2" gate="G$1" pin="SCL"/>
+<wire x1="55.88" y1="86.36" x2="55.88" y2="71.12" width="0.1524" layer="91"/>
+<junction x="55.88" y="71.12"/>
+</segment>
+</net>

Commit message: RDA5807 Arduino Library
Parts:
- added MUTE: (no value), adafruit:SWITCH_PUSHBUTTONC&K_KSS
Connections:
- new net N$3: MUTE.P$1, U2.PB3
- net GND: now also MUTE.P$2
Other:
- moved on the sheet: ANT1, CX1, CX2, J1
