File: extras/schematic/RDA5807FP_SETUP.sch (EAGLE design)
At the start: 17 parts, among them Q1 32768k, U1 ESP32-DEVKITC-32D, X1 HD44780LCD-1602

Commit message: RDA5807 Arduino Library
Parts:
- removed RDS_ON, SEEK, STEREO_MONO, VOL_DOWN, VOL_UP: (no value), adafruit:SWITCH_PUSHBUTTONC&K_KSS
- removed RE1: 62P16-H0, rotary-encoder:62P16-H0
- removed U1: ESP32-DEVKITC-32D, ESP32-DEVKITC-32D:ESP32-DEVKITC-32D
- removed VR1: 10k, SparkFun-Resistors:POTENTIOMETER-PTH-9MM-1/20W-20%
- removed X1: HD44780LCD-1602, adafruit:HD44780LCD-1602
Connections:
- removed net N$10: STEREO_MONO.P$2, U1.IO25
- removed net N$14: VR1.S, X1.VO
- removed net N$15: U1.IO18, X1.DB4
- removed net N$16: RE1.A
- removed net N$17: U1.IO17, X1.DB5
- removed net N$18: U1.IO16, X1.DB6
- removed net N$19: U1.IO15, X1.DB7
- removed net N$20: U1.IO32, VOL_UP.P$2
- removed net N$21: SEEK.P$2, U1.IO26
- removed net N$22: U1.IO33, VOL_DOWN.P$2
- removed net N$23: U1.IO19, X1.RS
- removed net N$24: U1.IO23, X1.E
- removed net VCC: VR1.E, X1.K
- removed net VSS: X1.RW, X1.VSS
- net GND: no longer RDS_ON.P$1, RE1.GND, SEEK.P$1, STEREO_MONO.P$1, U1.GND1, U1.GND3, VOL_DOWN.P$1, VOL_UP.P$1, VR1.A, X1.A
- net N$4: now also R1.1; no longer R2.1, U1.IO21
- net N$5: now also R2.1; no longer R1.1, U1.IO22
- net N$6: no longer U1.3V3
Other:
- note added: "SCLK/CLOCK"
- note added: "SDIO/SDA"
- note removed: "Encoder"
- note removed: "GPIO15"
- note removed: "GPIO16"
- note removed: "GPIO17"
- note removed: "GPIO18"
- note removed: "GPIO21 (SDA)"
- note removed: "GPIO22 (SCLK)"

Commit message: Documentation
Connections:
- net N$1: no longer R4.2
- net N$2: no longer R3.2
- net N$4: now also R4.2
- net N$5: now also R3.2
Other:
- moved on the sheet: R3, R4
Changed lines of the file:
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@@
 <text x="127" y="53.34" size="1.778" layer="91">RDA5807FP</text>
 <text x="162.56" y="15.24" size="1.778" layer="91">3.3V</text>
-<text x="114.3" y="-22.86" size="1.778" layer="91">I2C - PULLUP</text>
+<text x="99.06" y="-15.24" size="1.778" layer="91">I2C - PULLUP</text>
 <text x="172.72" y="35.56" size="1.778" layer="91">Audio Amp.</text>
-<text x="81.28" y="10.16" size="1.778" layer="91">SDIO/SDA</text>
-<text x="81.28" y="15.24" size="1.778" layer="91">SCLK/CLOCK</text>
+<text x="66.04" y="10.16" size="1.778" layer="91">SDIO/SDA</text>
+<text x="66.04" y="15.24" size="1.778" layer="91">SCLK/CLOCK</text>
 </plain>
 <instances>
@@
 <attribute name="VALUE" x="97.79" y="9.398" size="1.778" layer="96"/>
 </instance>
-<instance part="R3" gate="G$1" x="106.68" y="-7.62" smashed="yes" rot="R90">
-<attribute name="NAME" x="105.1814" y="-11.43" size="1.778" layer="95" rot="R90"/>
-<attribute name="VALUE" x="109.982" y="-11.43" size="1.778" layer="96" rot="R90"/>
-</instance>
-<instance part="R4" gate="G$1" x="116.84" y="-7.62" smashed="yes" rot="R90">
-<attribute name="NAME" x="115.3414" y="-11.43" size="1.778" layer="95" rot="R90"/>
-<attribute name="VALUE" x="120.142" y="-11.43" size="1.778" layer="96" rot="R90"/>
+<instance part="R3" gate="G$1" x="86.36" y="-7.62" smashed="yes" rot="R90">
+<attribute name="NAME" x="84.8614" y="-11.43" size="1.778" layer="95" rot="R90"/>
+<attribute name="VALUE" x="89.662" y="-11.43" size="1.778" layer="96" rot="R90"/>
+</instance>
+<instance part="R4" gate="G$1" x="93.98" y="-7.62" smashed="yes" rot="R90">
+<attribute name="NAME" x="92.4814" y="-11.43" size="1.778" layer="95" rot="R90"/>
+<attribute name="VALUE" x="97.282" y="-11.43" size="1.778" layer="96" rot="R90"/>
 </instance>
 <instance part="GND1" gate="1" x="111.76" y="38.1" smashed="yes">
@@
 <attribute name="C" x="106.68" y="48.26" size="1.778" layer="96"/>
 </instance>
-<instance part="GND7" gate="1" x="182.88" y="20.32" smashed="yes">
-<attribute name="VALUE" x="180.34" y="17.78" size="1.778" layer="96"/>
+<instance part="GND7" gate="1" x="185.42" y="20.32" smashed="yes">
+<attribute name="VALUE" x="182.88" y="17.78" size="1.778" layer="96"/>
 </instance>
 <instance part="C2" gate="G$1" x="160.02" y="33.02" smashed="yes" rot="R90">
@@
 <wire x1="152.4" y1="22.86" x2="172.72" y2="22.86" width="0.1524" layer="91"/>
 <pinref part="J1" gate="G$1" pin="SLEEVE"/>
-<wire x1="172.72" y1="22.86" x2="182.88" y2="22.86" width="0.1524" layer="91"/>
+<wire x1="172.72" y1="22.86" x2="185.42" y2="22.86" width="0.1524" layer="91"/>
 <wire x1="172.72" y1="27.94" x2="172.72" y2="22.86" width="0.1524" layer="91"/>
 <junction x="172.72" y="22.86"/>
@@
 <pinref part="U$1" gate="G$1" pin="SCLK"/>
 <wire x1="114.3" y1="17.78" x2="116.84" y2="17.78" width="0.1524" layer="91"/>
-<pinref part="R4" gate="G$1" pin="2"/>
-<wire x1="116.84" y1="-2.54" x2="116.84" y2="17.78" width="0.1524" layer="91"/>
-<junction x="116.84" y="17.78"/>
 </segment>
 </net>
@@
 <pinref part="U$1" gate="G$1" pin="SDA"/>
 <wire x1="106.68" y1="12.7" x2="116.84" y2="12.7" width="0.1524" layer="91"/>
-<pinref part="R3" gate="G$1" pin="2"/>
-<wire x1="106.68" y1="-2.54" x2="106.68" y2="12.7" width="0.1524" layer="91"/>
-<junction x="106.68" y="12.7"/>
-</segment>
-</net>
-<net name="N$6" class="0">
-<segment>
-<pinref part="R3" gate="G$1" pin="1"/>
-<pinref part="R4" gate="G$1" pin="1"/>
-<wire x1="106.68" y1="-12.7" x2="111.76" y2="-12.7" width="0.1524" layer="91"/>
-<wire x1="111.76" y1="-12.7" x2="116.84" y2="-12.7" width="0.1524" layer="91"/>
-<wire x1="111.76" y1="-30.48" x2="180.34" y2="-30.48" width="0.1524" layer="91"/>
-<wire x1="180.34" y1="-30.48" x2="180.34" y2="17.78" width="0.1524" layer="91"/>
-<pinref part="U$1" gate="G$1" pin="VDD"/>
-<wire x1="180.34" y1="17.78" x2="152.4" y2="17.78" width="0.1524" layer="91"/>
-<wire x1="111.76" y1="-12.7" x2="111.76" y2="-30.48" width="0.1524" layer="91"/>
-<junction x="111.76" y="-12.7"/>
 </segment>
 </net>
@@
 <segment>
 <pinref part="R1" gate="G$1" pin="1"/>
-<wire x1="104.14" y1="17.78" x2="86.36" y2="17.78" width="0.1524" layer="91"/>
-<junction x="86.36" y="17.78"/>
+<wire x1="104.14" y1="17.78" x2="93.98" y2="17.78" width="0.1524" layer="91"/>
+<junction x="81.28" y="17.78"/>
+<pinref part="R4" gate="G$1" pin="2"/>
+<wire x1="93.98" y1="17.78" x2="81.28" y2="17.78" width="0.1524" layer="91"/>
+<wire x1="93.98" y1="-2.54" x2="93.98" y2="17.78" width="0.1524" layer="91"/>
+<junction x="93.98" y="17.78"/>
 </segment>
 </net>
@@
 <pinref part="R2" gate="G$1" pin="1"/>
 <wire x1="96.52" y1="12.7" x2="86.36" y2="12.7" width="0.1524" layer="91"/>
+<junction x="81.28" y="12.7"/>
+<pinref part="R3" gate="G$1" pin="2"/>
+<wire x1="86.36" y1="12.7" x2="81.28" y2="12.7" width="0.1524" layer="91"/>
+<wire x1="86.36" y1="-2.54" x2="86.36" y2="12.7" width="0.1524" layer="91"/>
 <junction x="86.36" y="12.7"/>
 </segment>
 </net>
+<net name="N$10" class="0">
+<segment>
+<pinref part="R3" gate="G$1" pin="1"/>
+<pinref part="R4" gate="G$1" pin="1"/>
+<wire x1="86.36" y1="-12.7" x2="88.9" y2="-12.7" width="0.1524" layer="91"/>
+<wire x1="88.9" y1="-12.7" x2="93.98" y2="-12.7" width="0.1524" layer="91"/>
+<wire x1="88.9" y1="-12.7" x2="88.9" y2="-30.48" width="0.1524" layer="91"/>
+<junction x="88.9" y="-12.7"/>
+<wire x1="88.9" y1="-30.48" x2="180.34" y2="-30.48" width="0.1524" layer="91"/>
+<wire x1="180.34" y1="-30.48" x2="180.34" y2="17.78" width="0.1524" layer="91"/>
+<pinref part="U$1" gate="G$1" pin="VDD"/>
+<wire x1="180.34" y1="17.78" x2="152.4" y2="17.78" width="0.1524" layer="91"/>
+</segment>
+</net>

Commit message: RDA5807 Arduino Library
Other:
- note added: "RDA7088"
Changed lines of the file:
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@@
 <sheet>
 <plain>
-<text x="127" y="53.34" size="1.778" layer="91">RDA5807FP</text>
+<text x="124.46" y="55.88" size="1.778" layer="91">RDA5807FP</text>
 <text x="162.56" y="15.24" size="1.778" layer="91">3.3V</text>
 <text x="99.06" y="-15.24" size="1.778" layer="91">I2C - PULLUP</text>
@@
 <text x="66.04" y="10.16" size="1.778" layer="91">SDIO/SDA</text>
 <text x="66.04" y="15.24" size="1.778" layer="91">SCLK/CLOCK</text>
+<text x="124.46" y="53.34" size="1.778" layer="91">RDA7088</text>
 </plain>
 <instances>
